File: nuf5k-pcb.kicad_pcb (KiCad board)
At the start: 2 copper layers, 347.7 x 146.6 mm, 211 parts, among them J1 AVR-ISP-6, J2 1734366-1, J3 1734366-1, J4 1734366-1, SW0 KEYSW, SW1 KEYSW, SW10 KEYSW, SW11 KEYSW, SW12 KEYSW, SW16 KEYSW, SW17 KEYSW, SW18 KEYSW, SW19 KEYSW, SW2 KEYSW, SW20 KEYSW, SW21 KEYSW, SW22 KEYSW, SW23 KEYSW, SW24 KEYSW, SW25 KEYSW, SW26 KEYSW, SW27 KEYSW, SW28 KEYSW, SW29 KEYSW, SW3 KEYSW, SW30 KEYSW, SW31 KEYSW, SW33 KEYSW, SW34 KEYSW, SW35 KEYSW, SW36 KEYSW, SW37 KEYSW, SW38 KEYSW, SW39 KEYSW, SW4 KEYSW, SW40 KEYSW, SW41 KEYSW, SW42 KEYSW, SW43 KEYSW, SW44 KEYSW, SW45 KEYSW, SW46 KEYSW, SW47 KEYSW, SW48 KEYSW, SW5 KEYSW, SW50 KEYSW, SW51 KEYSW, SW52 KEYSW, SW53 KEYSW, SW54 KEYSW, SW55 KEYSW, SW56 KEYSW, SW57 KEYSW, SW58 KEYSW, SW59 KEYSW, SW6 KEYSW, SW60 KEYSW, SW61 KEYSW, SW62 KEYSW, SW63 KEYSW, SW64 KEYSW, SW65 KEYSW, SW66 KEYSW, SW67 KEYSW, SW68 KEYSW, SW69 KEYSW, SW7 KEYSW, SW70 KEYSW, SW71 KEYSW, SW72 KEYSW, SW73 KEYSW, SW74 KEYSW, SW75 KEYSW, SW76 KEYSW, SW77 KEYSW, SW78 KEYSW, SW79 KEYSW, SW8 KEYSW, SW80 KEYSW, SW81 KEYSW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

Commit message: added some usb stuff
Connections:
- J2 pad 5: unconnected-(J2-Pad5) -> (no net)
- J2 pad 6: unconnected-(J2-Pad6) -> (no net)
- J3 pad 5: unconnected-(J3-Pad5) -> (no net)
- J3 pad 6: unconnected-(J3-Pad6) -> (no net)
- J4 pad 5: unconnected-(J4-Pad5) -> (no net)
- J4 pad 6: unconnected-(J4-Pad6) -> (no net)
