File: nuf5k-pcb.kicad_sch (KiCad schematic)
At the start: 209 parts, among them J1 AVR-ISP-6, J2 1734366-1, J3 1734366-1, J4 1734366-1, SW0 KEYSW, SW1 KEYSW, SW10 KEYSW, SW11 KEYSW, SW12 KEYSW, SW13 KEYSW, SW14 KEYSW, SW15 KEYSW, SW16 KEYSW, SW17 KEYSW, SW18 KEYSW, SW19 KEYSW, SW2 KEYSW, SW20 KEYSW, SW21 KEYSW, SW22 KEYSW, SW23 KEYSW, SW24 KEYSW, SW25 KEYSW, SW26 KEYSW, SW27 KEYSW, SW28 KEYSW, SW29 KEYSW, SW3 KEYSW, SW30 KEYSW, SW31 KEYSW, SW32 KEYSW, SW33 KEYSW, SW34 KEYSW, SW35 KEYSW, SW36 KEYSW, SW37 KEYSW, SW38 KEYSW, SW39 KEYSW, SW4 KEYSW, SW40 KEYSW, SW41 KEYSW, SW42 KEYSW, SW43 KEYSW, SW44 KEYSW, SW45 KEYSW, SW46 KEYSW, SW47 KEYSW, SW48 KEYSW, SW49 KEYSW, SW5 KEYSW, SW50 KEYSW, SW51 KEYSW, SW52 KEYSW, SW53 KEYSW, SW54 KEYSW, SW55 KEYSW, SW56 KEYSW, SW57 KEYSW, SW58 KEYSW, SW59 KEYSW, SW6 KEYSW, SW60 KEYSW, SW61 KEYSW, SW62 KEYSW, SW63 KEYSW, SW64 KEYSW, SW65 KEYSW, SW66 KEYSW, SW67 KEYSW, SW68 KEYSW, SW69 KEYSW, SW7 KEYSW, SW70 KEYSW, SW71 KEYSW, SW72 KEYSW, SW73 KEYSW, SW74 KEYSW, SW75 KEYSW, SW76 KEYSW, SW77 KEYSW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

Commit message: added some usb stuff
Connections:
- net +5V: now also J2.1 (V+), J3.1 (V+), J4.1 (V+)
- net D+: now also U2.16 (DPU); no longer U1.16 (PD2)
- net D-: now also U2.15 (DMU); no longer U1.17 (PD3)
- net GND: now also J2.4 (GND), J3.4 (GND), J4.4 (GND), U2.1 (VSS)
- net at C2.1, Y1.2: now also U2.3 (XIN); no longer U1.12 (XTAL2)
- net at C1.1, Y1.1: now also U2.2 (XOUT); no longer U1.13 (XTAL1)
- net key_D-: now reaches U2.10 (DM1)
- net key_D-: now also U1.17 (PD3)
- net key_D+: now reaches U2.11 (DP1)
- net key_D+: now also U1.16 (PD2)
- net at U2.4 (DM4): now also J4.2 (D-)
- net at U2.5 (DP4): now also J4.3 (D+)
- net at U2.6 (DM3): now also J3.2 (D-)
- net at U2.7 (DP3): now also J3.3 (D+)
- net at U2.8 (DM2): now also J2.2 (D-)
- net at U2.9 (DP2): now also J2.3 (D+)
Other:
- note added: "https://electronics.stackexchange.com/questions/350140/how-can-i-add-additional-components-and-connections-to-make-this-usb-hub-functio"
- moved on the sheet: C1, C2, U2, Y1
